File: hardware/industrial-quad-relay.kicad_pcb (KiCad board)
At the start: 2 copper layers, 40 x 40 mm, 36 parts, among them P1 CON-SENSOR, P2 Digital Output, P3 Debug, P4 Boot, U1 XMC1XXX24, U2 CPC1020N, U3 CPC1020N, U4 CPC1020N, U5 CPC1020N, U6 DRILL, U7 DRILL, U8 DRILL, U9 DRILL

Commit message: specify processor
Parts:
- U1: value XMC1XXX24 -> XMC1100
Changed lines of the file:
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@@
       (effects (font (size 0.3 0.3) (thickness 0.075)))
     )
-    (fp_text value XMC1XXX24 (at 0 0.8 270) (layer F.Fab)
+    (fp_text value XMC1100 (at 0 0.8 270) (layer F.Fab)
       (effects (font (size 0.3 0.3) (thickness 0.075)))
     )
